File: PCB/i2c Board KiCad 6.kicad_pcb (KiCad board)
At the start: 2 copper layers, 19 parts, among them J1 SC-1 Expansion, J2 I2C Bus, J3 SPI BUS, J4 I2C_SEL, J5 SPI_SEL, J6 SPI_~{CS2}, J7 SPI_~{CS3}, J8 SPI_~{CS4}, J9 SPI_~{CS5}, U1 74HC138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

Commit message: Final Kicad PCB files complete
Parts:
- added Hole1: MountingHole_2.2mm_M2, MountingHole:MountingHole_2.2mm_M2, F.Cu at (126.0, 71.0)
- added Hole2: MountingHole_2.2mm_M2, MountingHole:MountingHole_2.2mm_M2, F.Cu at (186.0, 71.0)
- added Hole3: MountingHole_2.2mm_M2, MountingHole:MountingHole_2.2mm_M2, F.Cu at (126.0, 136.0)
- added Hole4: MountingHole_2.2mm_M2, MountingHole:MountingHole_2.2mm_M2, F.Cu at (186.0, 136.0)
- J6: value SPI_~{CS2} -> SPI~{CS2}
- J7: value SPI_~{CS3} -> SPI~{CS3}
- J8: value SPI_~{CS4} -> SPI~{CS4}
- J9: value SPI_~{CS5} -> SPI~{CS5}
- moved J3 61.6 mm to (128.5, 112.4)
- moved U5 50.4 mm to (164.2, 104.6)
- moved C2 45.6 mm to (165.5, 73.0)
- moved R3 39.2 mm to (138.2, 103.9), turned to 0 degrees
- moved U3 39.0 mm to (150.2, 81.4)
- moved J6 36.8 mm to (136.0, 74.0)
- moved J7 30.6 mm to (142.6, 74.0)
- moved J2 27.2 mm to (128.5, 84.5)
- moved R1 26.5 mm to (136.5, 84.2), turned to 0 degrees
- moved J8 25.4 mm to (149.6, 74.0)
- moved U4 24.7 mm to (137.1, 112.4)
- moved J9 24.2 mm to (156.6, 74.0)
- moved R2 22.6 mm to (136.5, 89.5), turned to 0 degrees
- moved U2 21.4 mm to (150.7, 112.4)
- moved J1 20.9 mm to (180.4, 79.4)
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Connections:
- J1 pad 10: /D5 -> /D6
- J1 pad 11: /D6 -> +5V
- J1 pad 12: +5V -> /D2
- J1 pad 13: /D2 -> /D7
- J1 pad 14: /D7 -> /D0
- J1 pad 15: /D0 -> /D1
- J1 pad 16: /D1 -> unconnected-(J1-Pad16)
- J1 pad 7: unconnected-(J1-Pad7) -> /D4
- J1 pad 8: /D4 -> /D3
- J1 pad 9: /D3 -> /D5
Routing:
- net Net-(J6-Pad1): track 0.00 -> 69.6 mm
- net Net-(J7-Pad1): track 0.00 -> 59.7 mm
- net Net-(J8-Pad1): track 0.00 -> 51.5 mm
- net /D3: track 25.5 -> 75.1 mm
- net GND: track 226.3 -> 180.7 mm
- net /A6: track 62.1 -> 19.7 mm
- net Net-(J9-Pad1): track 0.00 -> 39.5 mm
- net /A2: track 0.00 -> 38.5 mm
- net +5V: track 200.1 -> 164.7 mm
- net /A1: track 0.00 -> 35.3 mm
- net /A3: track 0.00 -> 33.0 mm
- net /D2: track 0.00 -> 33.0 mm
- net /~{IORQ}: track 25.5 -> 58.0 mm
- net /I2C_SDA: track 23.4 -> 55.7 mm
- net Net-(J5-Pad1): track 38.8 -> 71.0 mm, vias 0 -> 1
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Other:
- board outline added: 65.1 x 69.9 mm
- board text added: "+5v"
- board text added: "CLK"
- board text added: "D/~{C}"
- board text added: "GND"
- board text added: "MISO"
- board text added: "MOSI"
- board text added: "SCL"
- board text added: "SDA"
- board text added: "SPI2C board for SC-1 and TEC-1 Computers Designed by Craig Hart 2022 Revision 1"
- board text added: "~{CS}"
