File: PCB/i2c Board KiCad 6.kicad_sch (KiCad schematic)
At the start: 19 parts, among them J1 SC-1 Expansion, J2 I2C Bus, J3 SPI BUS, J4 I2C_SEL, J5 SPI_SEL, J6 SPI_~{CS2}, J7 SPI_~{CS3}, J8 SPI_~{CS4}, J9 SPI_~{CS5}, U1 74HC138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

Commit message: Final Kicad PCB files complete
Parts:
- J6: value SPI_~{CS2} -> SPI~{CS2}
- J7: value SPI_~{CS3} -> SPI~{CS3}
- J8: value SPI_~{CS4} -> SPI~{CS4}
- J9: value SPI_~{CS5} -> SPI~{CS5}
Connections:
- net +5V: now also J1.11 (Pin_11); no longer J1.12 (Pin_12)
- net D0: now also J1.14 (Pin_14); no longer J1.15 (Pin_15)
- net D1: now also J1.15 (Pin_15); no longer J1.16 (Pin_16)
- net D2: now also J1.12 (Pin_12); no longer J1.13 (Pin_13)
- net D3: now also J1.8 (Pin_8); no longer J1.9 (Pin_9)
- net D4: now also J1.7 (Pin_7); no longer J1.8 (Pin_8)
- net D5: now also J1.9 (Pin_9); no longer J1.10 (Pin_10)
- net D6: now also J1.10 (Pin_10); no longer J1.11 (Pin_11)
- net D7: now also J1.13 (Pin_13); no longer J1.14 (Pin_14)
Other:
- moved on the sheet: C1, C2
